Commit message: Fixes to ROS code for changes to API.

File: ROS/src/dogbot_description/urdf/dogbot.xacro (robot description, xacro)
@@ -6,5 +6,5 @@
   <xacro:property name="legoffset" value="0.125" />
   <xacro:property name="drivediam" value="0.08" />
-  <xacro:property name="upperleglen" value="0.36" />
+  <xacro:property name="upperleglen" value="0.30" />
   <xacro:property name="lowerleglen" value="0.31" />
   <xacro:property name="pi" value="3.1415" />

Commit message: Add method to drive the gazebo sim with the simple gait.

File: ROS/src/dogbot_description/urdf/dogbot.xacro (robot description, xacro)
@@ -8,4 +8,6 @@
   <xacro:property name="upperleglen" value="0.30" />
   <xacro:property name="lowerleglen" value="0.31" />
+  <xacro:property name="kp" value="1000000" />
+  <xacro:property name="kd" value="1.0" />
   <xacro:property name="pi" value="3.1415" />
   <material name="blue">
@@ -21,5 +23,5 @@
     <inertial>
       <mass value="${mass}" />
-      <inertia ixx="1.0" ixy="0.0" ixz="0.0" iyy="1.0" iyz="0.0" izz="1.0" />
+      <inertia ixx="0.2" ixy="0" ixz="0.0" iyy="0.2" iyz="0.0" izz="0.2" />
     </inertial>
   </xacro:macro>
@@ -38,5 +40,5 @@
       </geometry>
     </collision>
-    <xacro:default_inertial mass="4"/>
+    <xacro:default_inertial mass="6"/>
   </link>
   <joint name="base_joint" type="fixed">
@@ -48,6 +50,6 @@
     <mu1 value="200.0"/>
     <mu2 value="100.0"/>
-    <kp value="10000000.0" />
-    <kd value="1.0" />
+    <kp value="${kp}" />
+    <kd value="${kd}" />
     <material>Gazebo/white</material>
   </gazebo>
@@ -67,5 +69,5 @@
         </geometry>
       </collision>
-      <xacro:default_inertial mass="1"/>
+      <xacro:default_inertial mass="2"/>
     </link>
     <!--  -->
@@ -154,6 +156,6 @@
       <mu1 value="2000.0"/>
       <mu2 value="1000.0"/>
-      <kp value="10000000.0" />
-      <kd value="1.0" />
+      <kp value="${kp}" />
+      <kd value="${kd}" />
       <material>Gazebo/Grey</material>
     </gazebo>
@@ -175,4 +177,35 @@
          effort="500" velocity="10.0" />
     </joint>
+    <link name="${prefix}_${suffix}_foot">
+      <visual>
+        <origin xyz="0 0 0" rpy="${pi/2} 0 0" />
+        <geometry>
+          <!--cylinder radius="0.008" length="0.06"/-->
+          <sphere radius = "0.03"/>
+        </geometry>
+        <material name="black"/>
+      </visual>
+      <collision>
+        <origin xyz="0 0 0" rpy="${pi/2} 0 0" />
+        <geometry>
+          <!--cylinder radius="0.008" length="0.06"/-->
+          <sphere radius = "0.03"/>
+        </geometry>
+      </collision>
+      <xacro:default_inertial mass="0.0"/>
+    </link>
+    <joint name="${prefix}_${suffix}_foot_joint" type="fixed">
+      <axis xyz="0 1 0" rpy="0 0 0" />
+      <parent link="${prefix}_${suffix}_lowerleg"/>
+      <child link="${prefix}_${suffix}_foot"/>
+      <origin xyz="${lowerleglen * reflectx} 0 0" rpy="0 0 0"/>
+    </joint>
+    <gazebo reference="${prefix}_${suffix}_foot">
+      <mu1 value="2000000.0"/>
+      <mu2 value="1000000.0"/>
+      <kp value="${kp}" />
+      <kd value="${kd}" />
+      <material>Gazebo/Grey</material>
+    </gazebo>
     <transmission name="${prefix}_${suffix}_roll_transmition" >
       <type>transmission_interface/SimpleTransmission</type>

Commit message: Improve model, and correct the orientation of the joints.

File: ROS/src/dogbot_description/urdf/dogbot.xacro (robot description, xacro)
@@ -20,8 +20,16 @@
     <color rgba="1 1 1 1"/>
   </material>
-  <xacro:macro name="default_inertial" params="mass">
+  <xacro:macro name="default_inertial" params="mass xSize ySize zSize">
     <inertial>
       <mass value="${mass}" />
-      <inertia ixx="0.2" ixy="0" ixz="0.0" iyy="0.2" iyz="0.0" izz="0.2" />
+      <!-- Approximate mass distribution with a box -->
+      <inertia
+        ixx="${(1.0 / 12.0) * mass * (pow(ySize, 2) + pow(zSize, 2))}"
+        ixy="0"
+        ixz="0.0"
+        iyy="${(1.0 / 12.0) * mass * (pow(xSize, 2) + pow(zSize, 2))}"
+        iyz="0.0"
+        izz="${(1.0 / 12.0) * mass * (pow(xSize, 2) + pow(ySize, 2))}"
+      />
     </inertial>
   </xacro:macro>
@@ -40,5 +48,5 @@
       </geometry>
     </collision>
-    <xacro:default_inertial mass="6"/>
+    <xacro:default_inertial mass="6" xSize="${bodywidth}" ySize="${bodylen}" zSize="${bodyheight}" />
   </link>
   <joint name="base_joint" type="fixed">
@@ -69,5 +77,6 @@
         </geometry>
       </collision>
-      <xacro:default_inertial mass="2"/>
+      <!-- FIXME: check the location of center of mass. -->
+      <xacro:default_inertial mass="2.5" xSize="0.25" ySize="0.12" zSize="0.22"/>
     </link>
     <!--  -->
@@ -109,5 +118,5 @@
         </geometry>
       </collision>
-      <xacro:default_inertial mass="0.7"/>
+      <xacro:default_inertial mass="0.5" xSize="0.08" ySize="0.03" zSize="0.38" />
     </link>
     <joint name="${prefix}_${suffix}_pitch_joint" type="revolute">
@@ -151,5 +160,5 @@
         </geometry>
       </collision>
-      <xacro:default_inertial mass="0.3"/>
+      <xacro:default_inertial mass="0.2" xSize="0.03" ySize="0.02" zSize="0.36" />
     </link>
     <gazebo reference="${prefix}_${suffix}_lowerleg">
@@ -161,5 +170,5 @@
     </gazebo>
     <joint name="${prefix}_${suffix}_knee_joint" type="revolute">
-      <axis xyz="0 1 0" rpy="0 0 0" />
+      <axis xyz="0 -1 0" rpy="0 0 0" />
       <parent link="${prefix}_${suffix}_upperleg"/>
       <child link="${prefix}_${suffix}_lowerleg"/>
@@ -193,5 +202,5 @@
         </geometry>
       </collision>
-      <xacro:default_inertial mass="0.0"/>
+      <xacro:default_inertial mass="0.1" xSize="0.05" ySize="0.05" zSize="0.05"/>
     </link>
     <joint name="${prefix}_${suffix}_foot_joint" type="fixed">
